File: PCB/Macropad.kicad_pcb (KiCad board)
At the start: 2 copper layers, 67 x 85 mm, 21 parts, among them SW1 RotaryEncoder_Switch, SW10 SW_Push, SW2 SW_Push, SW3 SW_Push, SW4 SW_Push, SW5 SW_Push, SW6 SW_Push, SW7 SW_Push, SW8 SW_Push, SW9 SW_Push, U1 XIAO-RP2040-DIP

Commit message: Updated PCB
Connections:
- net C1 renamed col1
- net C2 renamed col2
- net C3 renamed col3
- net Net-(U1-GPIO29/ADC3/A3) renamed S1
- net Net-(U1-GPIO3/MOSI) renamed A
- net Net-(U1-GPIO4/MISO) renamed B
- net R3 renamed row3
- OLED1 pad 3: SCL -> Net-(OLED1-SCL)
- OLED1 pad 4: SDA -> Net-(OLED1-SDA)
- SW10 pad 2: R2 -> row2
- SW2 pad 2: R2 -> row2
- SW4 pad 2: R1 -> row1
- SW5 pad 2: R1 -> row1
- SW6 pad 2: R2 -> row2
- SW9 pad 2: R1 -> row1
- U1 pad 5: R2 -> Net-(OLED1-SDA)
- U1 pad 6: R1 -> Net-(OLED1-SCL)
- U1 pad 8: SCL -> row1
- U1 pad 9: SDA -> row2
Routing:
- net R2: track 93.7 -> 0.00 mm
- net row2: track 0.00 -> 81.3 mm
- net R1: track 69.4 -> 0.00 mm
- net row1: track 0.00 -> 56.5 mm
- net Net-(OLED1-SDA): track 0.00 -> 47.1 mm, vias 0 -> 1
- net Net-(OLED1-SCL): track 0.00 -> 41.6 mm
- net SCL: track 26.8 -> 0.00 mm
- net SDA: track 21.6 -> 0.00 mm
