File: PCB/Macropad.kicad_sch (KiCad schematic)
At the start: 21 parts, among them SW1 RotaryEncoder_Switch, SW10 SW_Push, SW2 SW_Push, SW3 SW_Push, SW4 SW_Push, SW5 SW_Push, SW6 SW_Push, SW7 SW_Push, SW8 SW_Push, SW9 SW_Push, U1 XIAO-RP2040-DIP

Commit message: Updated PCB
Connections:
- net row1: now also U1.8 (GPIO1/RX); no longer U1.6 (GPIO7/SCL)
- net row2: now also U1.9 (GPIO2/SCK); no longer U1.5 (GPIO6/SDA)
- net at OLED1.3 (SCL): now also U1.6 (GPIO7/SCL); no longer U1.8 (GPIO1/RX)
- net at OLED1.4 (SDA): now also U1.5 (GPIO6/SDA); no longer U1.9 (GPIO2/SCK)
Other:
- moved on the sheet: OLED1
Changed lines of the file:
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@@
 	(wire
 		(pts
-			(xy 151.13 130.81) (xy 162.56 130.81)
-		)
-		(stroke
-			(width 0)
-			(type default)
-		)
-	)
-	(wire
-		(pts
-			(xy 162.56 130.81) (xy 162.56 129.54)
+			(xy 78.74 119.38) (xy 71.12 119.38)
 		)
 		(stroke
@@
 	(wire
 		(pts
-			(xy 154.94 125.73) (xy 165.1 125.73)
+			(xy 73.66 127) (xy 57.15 127)
 		)
 		(stroke
@@
 	(wire
 		(pts
-			(xy 123.19 125.73) (xy 151.13 125.73)
-		)
-		(stroke
-			(width 0)
-			(type default)
-		)
-	)
-	(wire
-		(pts
 			(xy 199.39 72.39) (xy 224.79 72.39)
 		)
@@
 	(wire
 		(pts
+			(xy 57.15 123.19) (xy 71.12 123.19)
+		)
+		(stroke
+			(width 0)
+			(type default)
+		)
+	)
+	(wire
+		(pts
 			(xy 224.79 92.71) (xy 250.19 92.71)
 		)
@@
 	(wire
 		(pts
+			(xy 71.12 119.38) (xy 71.12 123.19)
+		)
+		(stroke
+			(width 0)
+			(type default)
+		)
+	)
+	(wire
+		(pts
 			(xy 181.61 33.02) (xy 181.61 54.61)
 		)
@@
 	(wire
 		(pts
-			(xy 165.1 118.11) (xy 149.86 118.11)
-		)
-		(stroke
-			(width 0)
-			(type default)
-		)
-	)
-	(wire
-		(pts
-			(xy 154.94 129.54) (xy 154.94 125.73)
+			(xy 57.15 115.57) (xy 72.39 115.57)
 		)
 		(stroke
@@
 	(wire
 		(pts
+			(xy 87.63 121.92) (xy 73.66 121.92)
+		)
+		(stroke
+			(width 0)
+			(type default)
+		)
+	)
+	(wire
+		(pts
 			(xy 232.41 48.26) (xy 232.41 67.31)
 		)
@@
 	(wire
 		(pts
-			(xy 123.19 129.54) (xy 154.94 129.54)
-		)
-		(stroke
-			(width 0)
-			(type default)
-		)
-	)
-	(wire
-		(pts
 			(xy 250.19 72.39) (xy 260.35 72.39)
 		)
@@
 	(wire
 		(pts
-			(xy 165.1 121.92) (xy 158.75 121.92)
+			(xy 57.15 119.38) (xy 63.5 119.38)
 		)
 		(stroke
@@
 	(wire
 		(pts
-			(xy 151.13 125.73) (xy 151.13 130.81)
-		)
-		(stroke
-			(width 0)
-			(type default)
-		)
-	)
-	(wire
-		(pts
 			(xy 199.39 92.71) (xy 224.79 92.71)
 		)
@@
 	(wire
 		(pts
-			(xy 162.56 129.54) (xy 165.1 129.54)
-		)
-		(stroke
-			(width 0)
-			(type default)
-		)
-	)
-	(wire
-		(pts
 			(xy 199.39 54.61) (xy 224.79 54.61)
 		)
@@
 	(wire
 		(pts
+			(xy 78.74 125.73) (xy 78.74 119.38)
+		)
+		(stroke
+			(width 0)
+			(type default)
+		)
+	)
+	(wire
+		(pts
 			(xy 232.41 34.29) (xy 232.41 48.26)
 		)
@@
 		(pts
 			(xy 250.19 67.31) (xy 250.19 72.39)
+		)
+		(stroke
+			(width 0)
+			(type default)
+		)
+	)
+	(wire
+		(pts
+			(xy 87.63 125.73) (xy 78.74 125.73)
+		)
+		(stroke
+			(width 0)
+			(type default)
+		)
+	)
+	(wire
+		(pts
+			(xy 73.66 121.92) (xy 73.66 127)
 		)
 		(stroke
@@
 	(global_label "row2"
 		(shape input)
-		(at 87.63 121.92 180)
+		(at 123.19 125.73 0)
 		(fields_autoplaced yes)
 		(effects
@@
 				(size 1.27 1.27)
 			)
-			(justify right)
+			(justify left)
 		)
 		(property "Intersheetrefs" "${INTERSHEET_REFS}"
-			(at 82.1653 121.92 0)
-			(hide yes)
-			(show_name no)
-			(do_not_autoplace no)
-			(effects
-				(font
-					(size 1.27 1.27)
-				)
-				(justify right)
+			(at 128.6547 125.73 0)
+			(hide yes)
+			(show_name no)
+			(do_not_autoplace no)
+			(effects
+				(font
+					(size 1.27 1.27)
+				)
+				(justify left)
 			)
 		)
@@
 	(global_label "row1"
 		(shape input)
-		(at 87.63 125.73 180)
+		(at 123.19 129.54 0)
 		(fields_autoplaced yes)
 		(effects
@@
 				(size 1.27 1.27)
 			)
-			(justify right)
+			(justify left)
 		)
 		(property "Intersheetrefs" "${INTERSHEET_REFS}"
-			(at 82.1653 125.73 0)
-			(hide yes)
-			(show_name no)
-			(do_not_autoplace no)
-			(effects
-				(font
-					(size 1.27 1.27)
-				)
-				(justify right)
+			(at 128.6547 129.54 0)
+			(hide yes)
+			(show_name no)
+			(do_not_autoplace no)
+			(effects
+				(font
+					(size 1.27 1.27)
+				)
+				(justify left)
 			)
 		)
@@
 	(symbol
 		(lib_id "screens for HACKpad:oled_1")
-		(at 166.37 123.19 0)
-		(mirror y)
+		(at 55.88 120.65 0)
 		(unit 1)
 		(body_style 1)
@@
 		(fields_autoplaced yes)
 		(property "Reference" "OLED1"
-			(at 179.705 111.76 0)
+			(at 42.545 109.22 0)
 			(show_name no)
 			(do_not_autoplace no)
@@
 		)
 		(property "Value" ""
-			(at 179.705 114.3 0)
+			(at 42.545 111.76 0)
 			(show_name no)
 			(do_not_autoplace no)
@@
 		)
 		(property "Footprint" ""
-			(at 166.37 123.19 0)
+			(at 55.88 120.65 0)
 			(hide yes)
 			(show_name no)
@@
 		)
 		(property "Datasheet" ""
-			(at 166.37 123.19 0)
+			(at 55.88 120.65 0)
 			(hide yes)
 			(show_name no)
@@
 		)
 		(property "Description" ""
-			(at 166.37 123.19 0)
+			(at 55.88 120.65 0)
 			(hide yes)
 			(show_name no)
@@
 	(symbol
 		(lib_id "power:GND")
-		(at 149.86 118.11 270)
-		(mirror x)
+		(at 72.39 115.57 90)
 		(unit 1)
 		(body_style 1)
@@
 		(fields_autoplaced yes)
 		(property "Reference" "#PWR05"
-			(at 143.51 118.11 0)
+			(at 78.74 115.57 0)
 			(hide yes)
 			(show_name no)
@@
 		)
 		(property "Value" "GND"
-			(at 148.59 114.3 90)
+			(at 73.66 111.76 90)
 			(show_name no)
 			(do_not_autoplace no)
@@
 		)
 		(property "Footprint" ""
-			(at 149.86 118.11 0)
+			(at 72.39 115.57 0)
 			(hide yes)
 			(show_name no)
@@
 		)
 		(property "Datasheet" ""
-			(at 149.86 118.11 0)
+			(at 72.39 115.57 0)
 			(hide yes)
 			(show_name no)
@@
 		)
 		(property "Description" "Power symbol creates a global label with name \"GND\" , ground"
-			(at 149.86 118.11 0)
+			(at 72.39 115.57 0)
 			(hide yes)
 			(show_name no)
@@
 	(symbol
 		(lib_id "power:+3V3")
-		(at 158.75 121.92 90)
-		(mirror x)
+		(at 63.5 119.38 270)
 		(unit 1)
 		(body_style 1)
@@
 		(fields_autoplaced yes)
 		(property "Reference" "#PWR06"
-			(at 162.56 121.92 0)
+			(at 59.69 119.38 0)
 			(hide yes)
 			(show_name no)
@@
 		)
 		(property "Value" "+3V3"
-			(at 157.48 119.38 90)
+			(at 64.77 116.84 90)
 			(show_name no)
 			(do_not_autoplace no)
@@
 		)
 		(property "Footprint" ""
-			(at 158.75 121.92 0)
+			(at 63.5 119.38 0)
 			(hide yes)
 			(show_name no)
@@
 		)
 		(property "Datasheet" ""
-			(at 158.75 121.92 0)
+			(at 63.5 119.38 0)
 			(hide yes)
 			(show_name no)
@@
 		)
 		(property "Description" "Power symbol creates a global label with name \"+3V3\""
-			(at 158.75 121.92 0)
-			(hide yes)
-			(show_name no)
+			(at 63.5 119.38 0)
+			(hide yes)
+			(show_name no)
